Commit message: complete the new env wrapper but with bugs to fix

File: assets/robot/hexapod_34/urdf/hexapod_34.urdf (robot description, URDF)
Before this commit: robot hexapod_34, 19 links, 18 joints
Joints:
- joint l1_bc: axis 0 0 -1 -> 0 0 1
- joint l2_bc: axis 0 0 -1 -> 0 0 1
- joint l3_bc: axis 0 0 -1 -> 0 0 1
- joint r1_bc: axis 0 0 -1 -> 0 0 1
- joint r1_cf: axis 0 0 1 -> 0 0 -1
- joint r1_ft: axis 0 0 1 -> 0 0 -1
- joint r2_bc: axis 0 0 -1 -> 0 0 1
- joint r2_cf: axis 0 0 1 -> 0 0 -1
- joint r2_ft: axis 0 0 1 -> 0 0 -1
- joint r3_bc: axis 0 0 -1 -> 0 0 1
- joint r3_cf: axis 0 0 1 -> 0 0 -1
- joint r3_ft: axis 0 1.9702E-05 1 -> 0 0 -1

Commit message: revise the hip direction of the left legs

File: assets/robot/hexapod_34/urdf/hexapod_34.urdf (robot description, URDF)
Before this commit: robot hexapod_34, 19 links, 18 joints
Joints:
- joint l1_bc: axis 0 0 1 -> 0 0 -1
- joint l2_bc: axis 0 0 1 -> 0 0 -1
- joint l3_bc: axis 0 0 1 -> 0 0 -1

Commit message: modify the urdf for the orientation as loaded

File: assets/robot/hexapod_34/urdf/hexapod_34.urdf (robot description, URDF)
Before this commit: robot hexapod_34, 19 links, 18 joints
Links:
- added link rotated_base, mass 1.0
Joints:
- added joint rotate_base: type fixed, parent rotated_base, child base_link, origin xyz=0 0 0 rpy=0 0 -1.5708
