Commit message: modify ground for training

File: assets/custom_ground.urdf (robot description, URDF)
Before this commit: robot random_terrain, 101 links, 100 joints
Links:
- link tile_0_0: geometry collision box size=0.5 0.5 0.0283; visual box size=0.5 0.5 0.0283
- link tile_0_1: geometry collision box size=0.5 0.5 0.0228; visual box size=0.5 0.5 0.0228
- link tile_0_2: geometry collision box size=0.5 0.5 0.0268; visual box size=0.5 0.5 0.0268
- link tile_0_3: geometry collision box size=0.5 0.5 0.0136; visual box size=0.5 0.5 0.0136
- link tile_0_4: geometry collision box size=0.5 0.5 0.0257; visual box size=0.5 0.5 0.0257
- link tile_0_5: geometry collision box size=0.5 0.5 0.0231; visual box size=0.5 0.5 0.0231
- link tile_0_6: geometry collision box size=0.5 0.5 0.0373; visual box size=0.5 0.5 0.0373
- link tile_0_7: geometry collision box size=0.5 0.5 0.0286; visual box size=0.5 0.5 0.0286
- link tile_0_8: geometry collision box size=0.5 0.5 0.0141; visual box size=0.5 0.5 0.0141
- link tile_0_9: geometry collision box size=0.5 0.5 0.0117; visual box size=0.5 0.5 0.0117
- link tile_1_0: geometry collision box size=0.5 0.5 0.0310; visual box size=0.5 0.5 0.0310
- link tile_1_1: geometry collision box size=0.5 0.5 0.0266; visual box size=0.5 0.5 0.0266
- link tile_1_2: geometry collision box size=0.5 0.5 0.0386; visual box size=0.5 0.5 0.0386
- link tile_1_3: geometry collision box size=0.5 0.5 0.0319; visual box size=0.5 0.5 0.0319
- link tile_1_4: geometry collision box size=0.5 0.5 0.0356; visual box size=0.5 0.5 0.0356
- link tile_1_5: geometry collision box size=0.5 0.5 0.0257; visual box size=0.5 0.5 0.0257
- link tile_1_6: geometry collision box size=0.5 0.5 0.0351; visual box size=0.5 0.5 0.0351
- link tile_1_7: geometry collision box size=0.5 0.5 0.0208; visual box size=0.5 0.5 0.0208
- link tile_1_8: geometry collision box size=0.5 0.5 0.0246; visual box size=0.5 0.5 0.0246
- link tile_1_9: geometry collision box size=0.5 0.5 0.0238; visual box size=0.5 0.5 0.0238
- link tile_2_0: geometry collision box size=0.5 0.5 0.0302; visual box size=0.5 0.5 0.0302
- link tile_2_1: geometry collision box size=0.5 0.5 0.0280; visual box size=0.5 0.5 0.0280
- link tile_2_2: geometry collision box size=0.5 0.5 0.0313; visual box size=0.5 0.5 0.0313
- link tile_2_3: geometry collision box size=0.5 0.5 0.0306; visual box size=0.5 0.5 0.0306
- link tile_2_4: geometry collision box size=0.5 0.5 0.0352; visual box size=0.5 0.5 0.0352
- link tile_2_5: geometry collision box size=0.5 0.5 0.0381; visual box size=0.5 0.5 0.0381
- link tile_2_6: geometry collision box size=0.5 0.5 0.0207; visual box size=0.5 0.5 0.0207
- link tile_2_7: geometry collision box size=0.5 0.5 0.0161; visual box size=0.5 0.5 0.0161
- link tile_2_8: geometry collision box size=0.5 0.5 0.0386; visual box size=0.5 0.5 0.0386
- link tile_2_9: geometry collision box size=0.5 0.5 0.0180; visual box size=0.5 0.5 0.0180
- link tile_3_0: geometry collision box size=0.5 0.5 0.0366; visual box size=0.5 0.5 0.0366
- link tile_3_1: geometry collision box size=0.5 0.5 0.0280; visual box size=0.5 0.5 0.0280
- link tile_3_2: geometry collision box size=0.5 0.5 0.0357; visual box size=0.5 0.5 0.0357
- link tile_3_3: geometry collision box size=0.5 0.5 0.0306; visual box size=0.5 0.5 0.0306
- link tile_3_4: geometry collision box size=0.5 0.5 0.0237; visual box size=0.5 0.5 0.0237
- link tile_3_5: geometry collision box size=0.5 0.5 0.0328; visual box size=0.5 0.5 0.0328
- link tile_3_6: geometry collision box size=0.5 0.5 0.0205; visual box size=0.5 0.5 0.0205
- link tile_3_7: geometry collision box size=0.5 0.5 0.0370; visual box size=0.5 0.5 0.0370
- link tile_3_8: geometry collision box size=0.5 0.5 0.0274; visual box size=0.5 0.5 0.0274
- link tile_3_9: geometry collision box size=0.5 0.5 0.0296; visual box size=0.5 0.5 0.0296
- link tile_4_0: geometry collision box size=0.5 0.5 0.0293; visual box size=0.5 0.5 0.0293
- link tile_4_1: geometry collision box size=0.5 0.5 0.0317; visual box size=0.5 0.5 0.0317
- link tile_4_2: geometry collision box size=0.5 0.5 0.0270; visual box size=0.5 0.5 0.0270
- link tile_4_3: geometry collision box size=0.5 0.5 0.0273; visual box size=0.5 0.5 0.0273
- link tile_4_4: geometry collision box size=0.5 0.5 0.0156; visual box size=0.5 0.5 0.0156
- link tile_4_5: geometry collision box size=0.5 0.5 0.0213; visual box size=0.5 0.5 0.0213
- link tile_4_6: geometry collision box size=0.5 0.5 0.0126; visual box size=0.5 0.5 0.0126
- link tile_4_7: geometry collision box size=0.5 0.5 0.0397; visual box size=0.5 0.5 0.0397
- link tile_4_8: geometry collision box size=0.5 0.5 0.0347; visual box size=0.5 0.5 0.0347
- link tile_4_9: geometry collision box size=0.5 0.5 0.0109; visual box size=0.5 0.5 0.0109
- link tile_5_0: geometry collision box size=0.5 0.5 0.0384; visual box size=0.5 0.5 0.0384
- link tile_5_1: geometry collision box size=0.5 0.5 0.0275; visual box size=0.5 0.5 0.0275
- link tile_5_2: geometry collision box size=0.5 0.5 0.0135; visual box size=0.5 0.5 0.0135
- link tile_5_3: geometry collision box size=0.5 0.5 0.0103; visual box size=0.5 0.5 0.0103
- link tile_5_4: geometry collision box size=0.5 0.5 0.0352; visual box size=0.5 0.5 0.0352
- link tile_5_5: geometry collision box size=0.5 0.5 0.0156; visual box size=0.5 0.5 0.0156
- link tile_5_6: geometry collision box size=0.5 0.5 0.0354; visual box size=0.5 0.5 0.0354
- link tile_5_7: geometry collision box size=0.5 0.5 0.0207; visual box size=0.5 0.5 0.0207
- link tile_5_8: geometry collision box size=0.5 0.5 0.0123; visual box size=0.5 0.5 0.0123
- link tile_5_9: geometry collision box size=0.5 0.5 0.0383; visual box size=0.5 0.5 0.0383
- link tile_6_0: geometry collision box size=0.5 0.5 0.0119; visual box size=0.5 0.5 0.0119
- link tile_6_1: geometry collision box size=0.5 0.5 0.0108; visual box size=0.5 0.5 0.0108
- link tile_6_2: geometry collision box size=0.5 0.5 0.0350; visual box size=0.5 0.5 0.0350
- link tile_6_3: geometry collision box size=0.5 0.5 0.0346; visual box size=0.5 0.5 0.0346
- link tile_6_4: geometry collision box size=0.5 0.5 0.0265; visual box size=0.5 0.5 0.0265
- link tile_6_5: geometry collision box size=0.5 0.5 0.0304; visual box size=0.5 0.5 0.0304
- link tile_6_6: geometry collision box size=0.5 0.5 0.0144; visual box size=0.5 0.5 0.0144
- link tile_6_7: geometry collision box size=0.5 0.5 0.0289; visual box size=0.5 0.5 0.0289
- link tile_6_8: geometry collision box size=0.5 0.5 0.0196; visual box size=0.5 0.5 0.0196
- link tile_6_9: geometry collision box size=0.5 0.5 0.0112; visual box size=0.5 0.5 0.0112
- link tile_7_0: geometry collision box size=0.5 0.5 0.0115; visual box size=0.5 0.5 0.0115
- link tile_7_1: geometry collision box size=0.5 0.5 0.0315; visual box size=0.5 0.5 0.0315
- link tile_7_2: geometry collision box size=0.5 0.5 0.0348; visual box size=0.5 0.5 0.0348
- link tile_7_3: geometry collision box size=0.5 0.5 0.0204; visual box size=0.5 0.5 0.0204
- link tile_7_4: geometry collision box size=0.5 0.5 0.0337; visual box size=0.5 0.5 0.0337
- link tile_7_5: geometry collision box size=0.5 0.5 0.0157; visual box size=0.5 0.5 0.0157
- link tile_7_6: geometry collision box size=0.5 0.5 0.0194; visual box size=0.5 0.5 0.0194
- link tile_7_7: geometry collision box size=0.5 0.5 0.0126; visual box size=0.5 0.5 0.0126
- link tile_7_8: geometry collision box size=0.5 0.5 0.0355; visual box size=0.5 0.5 0.0355
- link tile_7_9: geometry collision box size=0.5 0.5 0.0340; visual box size=0.5 0.5 0.0340
- link tile_8_0: geometry collision box size=0.5 0.5 0.0391; visual box size=0.5 0.5 0.0391
- link tile_8_1: geometry collision box size=0.5 0.5 0.0154; visual box size=0.5 0.5 0.0154
- link tile_8_2: geometry collision box size=0.5 0.5 0.0267; visual box size=0.5 0.5 0.0267
- link tile_8_3: geometry collision box size=0.5 0.5 0.0291; visual box size=0.5 0.5 0.0291
- link tile_8_4: geometry collision box size=0.5 0.5 0.0321; visual box size=0.5 0.5 0.0321
- link tile_8_5: geometry collision box size=0.5 0.5 0.0157; visual box size=0.5 0.5 0.0157
- link tile_8_6: geometry collision box size=0.5 0.5 0.0224; visual box size=0.5 0.5 0.0224
- link tile_8_7: geometry collision box size=0.5 0.5 0.0193; visual box size=0.5 0.5 0.0193
- link tile_8_8: geometry collision box size=0.5 0.5 0.0163; visual box size=0.5 0.5 0.0163
- link tile_8_9: geometry collision box size=0.5 0.5 0.0230; visual box size=0.5 0.5 0.0230
- link tile_9_0: geometry collision box size=0.5 0.5 0.0113; visual box size=0.5 0.5 0.0113
- link tile_9_1: geometry collision box size=0.5 0.5 0.0130; visual box size=0.5 0.5 0.0130
- link tile_9_2: geometry collision box size=0.5 0.5 0.0155; visual box size=0.5 0.5 0.0155
- link tile_9_3: geometry collision box size=0.5 0.5 0.0224; visual box size=0.5 0.5 0.0224
- link tile_9_4: geometry collision box size=0.5 0.5 0.0121; visual box size=0.5 0.5 0.0121
- link tile_9_5: geometry collision box size=0.5 0.5 0.0382; visual box size=0.5 0.5 0.0382
- link tile_9_6: geometry collision box size=0.5 0.5 0.0187; visual box size=0.5 0.5 0.0187
- link tile_9_7: geometry collision box size=0.5 0.5 0.0347; visual box size=0.5 0.5 0.0347
- link tile_9_8: geometry collision box size=0.5 0.5 0.0217; visual box size=0.5 0.5 0.0217
- link tile_9_9: geometry collision box size=0.5 0.5 0.0232; visual box size=0.5 0.5 0.0232
Joints:
- joint joint_tile_0_0: origin xyz=-1.350 -1.350 0.013 rpy=0 0 0 -> xyz=-2.250 -2.250 0.014 rpy=0 0 0
- joint joint_tile_0_1: origin xyz=-1.050 -1.350 0.030 rpy=0 0 0 -> xyz=-1.750 -2.250 0.011 rpy=0 0 0
- joint joint_tile_0_2: origin xyz=-0.750 -1.350 0.009 rpy=0 0 0 -> xyz=-1.250 -2.250 0.013 rpy=0 0 0
- joint joint_tile_0_3: origin xyz=-0.450 -1.350 0.023 rpy=0 0 0 -> xyz=-0.750 -2.250 0.007 rpy=0 0 0
- joint joint_tile_0_4: origin xyz=-0.150 -1.350 0.012 rpy=0 0 0 -> xyz=-0.250 -2.250 0.013 rpy=0 0 0
- joint joint_tile_0_5: origin xyz=0.150 -1.350 0.029 rpy=0 0 0 -> xyz=0.250 -2.250 0.012 rpy=0 0 0
- joint joint_tile_0_6: origin xyz=0.450 -1.350 0.018 rpy=0 0 0 -> xyz=0.750 -2.250 0.019 rpy=0 0 0
- joint joint_tile_0_7: origin xyz=0.750 -1.350 0.028 rpy=0 0 0 -> xyz=1.250 -2.250 0.014 rpy=0 0 0
- joint joint_tile_0_8: origin xyz=1.050 -1.350 0.030 rpy=0 0 0 -> xyz=1.750 -2.250 0.007 rpy=0 0 0
- joint joint_tile_0_9: origin xyz=1.350 -1.350 0.018 rpy=0 0 0 -> xyz=2.250 -2.250 0.006 rpy=0 0 0
- joint joint_tile_1_0: origin xyz=-1.350 -1.050 0.033 rpy=0 0 0 -> xyz=-2.250 -1.750 0.016 rpy=0 0 0
- joint joint_tile_1_1: origin xyz=-1.050 -1.050 0.011 rpy=0 0 0 -> xyz=-1.750 -1.750 0.013 rpy=0 0 0
- joint joint_tile_1_2: origin xyz=-0.750 -1.050 0.031 rpy=0 0 0 -> xyz=-1.250 -1.750 0.019 rpy=0 0 0
- joint joint_tile_1_3: origin xyz=-0.450 -1.050 0.025 rpy=0 0 0 -> xyz=-0.750 -1.750 0.016 rpy=0 0 0
- joint joint_tile_1_4: origin xyz=-0.150 -1.050 0.016 rpy=0 0 0 -> xyz=-0.250 -1.750 0.018 rpy=0 0 0
- joint joint_tile_1_5: origin xyz=0.150 -1.050 0.025 rpy=0 0 0 -> xyz=0.250 -1.750 0.013 rpy=0 0 0
- joint joint_tile_1_6: origin xyz=0.450 -1.050 0.012 rpy=0 0 0 -> xyz=0.750 -1.750 0.018 rpy=0 0 0
- joint joint_tile_1_7: origin xyz=0.750 -1.050 0.008 rpy=0 0 0 -> xyz=1.250 -1.750 0.010 rpy=0 0 0
- joint joint_tile_1_8: origin xyz=1.050 -1.050 0.029 rpy=0 0 0 -> xyz=1.750 -1.750 0.012 rpy=0 0 0
- joint joint_tile_1_9: origin xyz=1.350 -1.050 0.010 rpy=0 0 0 -> xyz=2.250 -1.750 0.012 rpy=0 0 0
- joint joint_tile_2_0: origin xyz=-1.350 -0.750 0.012 rpy=0 0 0 -> xyz=-2.250 -1.250 0.015 rpy=0 0 0
- joint joint_tile_2_1: origin xyz=-1.050 -0.750 0.008 rpy=0 0 0 -> xyz=-1.750 -1.250 0.014 rpy=0 0 0
- joint joint_tile_2_2: origin xyz=-0.750 -0.750 0.012 rpy=0 0 0 -> xyz=-1.250 -1.250 0.016 rpy=0 0 0
- joint joint_tile_2_3: origin xyz=-0.450 -0.750 0.033 rpy=0 0 0 -> xyz=-0.750 -1.250 0.015 rpy=0 0 0
- joint joint_tile_2_4: origin xyz=-0.150 -0.750 0.014 rpy=0 0 0 -> xyz=-0.250 -1.250 0.018 rpy=0 0 0
- joint joint_tile_2_5: origin xyz=0.150 -0.750 0.035 rpy=0 0 0 -> xyz=0.250 -1.250 0.019 rpy=0 0 0
- joint joint_tile_2_6: origin xyz=0.450 -0.750 0.031 rpy=0 0 0 -> xyz=0.750 -1.250 0.010 rpy=0 0 0
- joint joint_tile_2_7: origin xyz=0.750 -0.750 0.014 rpy=0 0 0 -> xyz=1.250 -1.250 0.008 rpy=0 0 0
- joint joint_tile_2_8: origin xyz=1.050 -0.750 0.011 rpy=0 0 0 -> xyz=1.750 -1.250 0.019 rpy=0 0 0
- joint joint_tile_2_9: origin xyz=1.350 -0.750 0.008 rpy=0 0 0 -> xyz=2.250 -1.250 0.009 rpy=0 0 0
- joint joint_tile_3_0: origin xyz=-1.350 -0.450 0.025 rpy=0 0 0 -> xyz=-2.250 -0.750 0.018 rpy=0 0 0
- joint joint_tile_3_1: origin xyz=-1.050 -0.450 0.007 rpy=0 0 0 -> xyz=-1.750 -0.750 0.014 rpy=0 0 0
- joint joint_tile_3_2: origin xyz=-0.750 -0.450 0.017 rpy=0 0 0 -> xyz=-1.250 -0.750 0.018 rpy=0 0 0
- joint joint_tile_3_3: origin xyz=-0.450 -0.450 0.015 rpy=0 0 0 -> xyz=-0.750 -0.750 0.015 rpy=0 0 0
- joint joint_tile_3_4: origin xyz=-0.150 -0.450 0.029 rpy=0 0 0 -> xyz=-0.250 -0.750 0.012 rpy=0 0 0
- joint joint_tile_3_5: origin xyz=0.150 -0.450 0.005 rpy=0 0 0 -> xyz=0.250 -0.750 0.016 rpy=0 0 0
- joint joint_tile_3_6: origin xyz=0.450 -0.450 0.017 rpy=0 0 0 -> xyz=0.750 -0.750 0.010 rpy=0 0 0
- joint joint_tile_3_7: origin xyz=0.750 -0.450 0.030 rpy=0 0 0 -> xyz=1.250 -0.750 0.018 rpy=0 0 0
- joint joint_tile_3_8: origin xyz=1.050 -0.450 0.026 rpy=0 0 0 -> xyz=1.750 -0.750 0.014 rpy=0 0 0
- joint joint_tile_3_9: origin xyz=1.350 -0.450 0.029 rpy=0 0 0 -> xyz=2.250 -0.750 0.015 rpy=0 0 0
- joint joint_tile_4_0: origin xyz=-1.350 -0.150 0.012 rpy=0 0 0 -> xyz=-2.250 -0.250 0.015 rpy=0 0 0
- joint joint_tile_4_1: origin xyz=-1.050 -0.150 0.020 rpy=0 0 0 -> xyz=-1.750 -0.250 0.016 rpy=0 0 0
- joint joint_tile_4_2: origin xyz=-0.750 -0.150 0.028 rpy=0 0 0 -> xyz=-1.250 -0.250 0.014 rpy=0 0 0
- joint joint_tile_4_3: origin xyz=-0.450 -0.150 0.033 rpy=0 0 0 -> xyz=-0.750 -0.250 0.014 rpy=0 0 0
- joint joint_tile_4_4: origin xyz=-0.150 -0.150 0.032 rpy=0 0 0 -> xyz=-0.250 -0.250 0.008 rpy=0 0 0
- joint joint_tile_4_5: origin xyz=0.150 -0.150 0.022 rpy=0 0 0 -> xyz=0.250 -0.250 0.011 rpy=0 0 0
- joint joint_tile_4_6: origin xyz=0.450 -0.150 0.017 rpy=0 0 0 -> xyz=0.750 -0.250 0.006 rpy=0 0 0
- joint joint_tile_4_7: origin xyz=0.750 -0.150 0.014 rpy=0 0 0 -> xyz=1.250 -0.250 0.020 rpy=0 0 0
- joint joint_tile_4_8: origin xyz=1.050 -0.150 0.015 rpy=0 0 0 -> xyz=1.750 -0.250 0.017 rpy=0 0 0
- joint joint_tile_4_9: origin xyz=1.350 -0.150 0.021 rpy=0 0 0 -> xyz=2.250 -0.250 0.005 rpy=0 0 0
- joint joint_tile_5_0: origin xyz=-1.350 0.150 0.012 rpy=0 0 0 -> xyz=-2.250 0.250 0.019 rpy=0 0 0
- joint joint_tile_5_1: origin xyz=-1.050 0.150 0.014 rpy=0 0 0 -> xyz=-1.750 0.250 0.014 rpy=0 0 0
- joint joint_tile_5_2: origin xyz=-0.750 0.150 0.025 rpy=0 0 0 -> xyz=-1.250 0.250 0.007 rpy=0 0 0
- joint joint_tile_5_3: origin xyz=-0.450 0.150 0.012 rpy=0 0 0 -> xyz=-0.750 0.250 0.005 rpy=0 0 0
- joint joint_tile_5_4: origin xyz=-0.150 0.150 0.029 rpy=0 0 0 -> xyz=-0.250 0.250 0.018 rpy=0 0 0
- joint joint_tile_5_5: origin xyz=0.150 0.150 0.021 rpy=0 0 0 -> xyz=0.250 0.250 0.008 rpy=0 0 0
- joint joint_tile_5_6: origin xyz=0.450 0.150 0.029 rpy=0 0 0 -> xyz=0.750 0.250 0.018 rpy=0 0 0
- joint joint_tile_5_7: origin xyz=0.750 0.150 0.025 rpy=0 0 0 -> xyz=1.250 0.250 0.010 rpy=0 0 0
- joint joint_tile_5_8: origin xyz=1.050 0.150 0.009 rpy=0 0 0 -> xyz=1.750 0.250 0.006 rpy=0 0 0
- joint joint_tile_5_9: origin xyz=1.350 0.150 0.029 rpy=0 0 0 -> xyz=2.250 0.250 0.019 rpy=0 0 0
- joint joint_tile_6_0: origin xyz=-1.350 0.450 0.019 rpy=0 0 0 -> xyz=-2.250 0.750 0.006 rpy=0 0 0
- joint joint_tile_6_1: origin xyz=-1.050 0.450 0.027 rpy=0 0 0 -> xyz=-1.750 0.750 0.005 rpy=0 0 0
- joint joint_tile_6_2: origin xyz=-0.750 0.450 0.010 rpy=0 0 0 -> xyz=-1.250 0.750 0.017 rpy=0 0 0
- joint joint_tile_6_3: origin xyz=-0.450 0.450 0.027 rpy=0 0 0 -> xyz=-0.750 0.750 0.017 rpy=0 0 0
- joint joint_tile_6_4: origin xyz=-0.150 0.450 0.015 rpy=0 0 0 -> xyz=-0.250 0.750 0.013 rpy=0 0 0
- joint joint_tile_6_5: origin xyz=0.150 0.450 0.009 rpy=0 0 0 -> xyz=0.250 0.750 0.015 rpy=0 0 0
- joint joint_tile_6_6: origin xyz=0.450 0.450 0.018 rpy=0 0 0 -> xyz=0.750 0.750 0.007 rpy=0 0 0
- joint joint_tile_6_7: origin xyz=0.750 0.450 0.030 rpy=0 0 0 -> xyz=1.250 0.750 0.014 rpy=0 0 0
- joint joint_tile_6_8: origin xyz=1.050 0.450 0.017 rpy=0 0 0 -> xyz=1.750 0.750 0.010 rpy=0 0 0
- joint joint_tile_6_9: origin xyz=1.350 0.450 0.026 rpy=0 0 0 -> xyz=2.250 0.750 0.006 rpy=0 0 0
- joint joint_tile_7_0: origin xyz=-1.350 0.750 0.027 rpy=0 0 0 -> xyz=-2.250 1.250 0.006 rpy=0 0 0
- joint joint_tile_7_1: origin xyz=-1.050 0.750 0.028 rpy=0 0 0 -> xyz=-1.750 1.250 0.016 rpy=0 0 0
- joint joint_tile_7_2: origin xyz=-0.750 0.750 0.013 rpy=0 0 0 -> xyz=-1.250 1.250 0.017 rpy=0 0 0
- joint joint_tile_7_3: origin xyz=-0.450 0.750 0.029 rpy=0 0 0 -> xyz=-0.750 1.250 0.010 rpy=0 0 0
- joint joint_tile_7_4: origin xyz=-0.150 0.750 0.035 rpy=0 0 0 -> xyz=-0.250 1.250 0.017 rpy=0 0 0
- joint joint_tile_7_5: origin xyz=0.150 0.750 0.011 rpy=0 0 0 -> xyz=0.250 1.250 0.008 rpy=0 0 0
- joint joint_tile_7_6: origin xyz=0.450 0.750 0.021 rpy=0 0 0 -> xyz=0.750 1.250 0.010 rpy=0 0 0
- joint joint_tile_7_7: origin xyz=0.750 0.750 0.018 rpy=0 0 0 -> xyz=1.250 1.250 0.006 rpy=0 0 0
- joint joint_tile_7_8: origin xyz=1.050 0.750 0.009 rpy=0 0 0 -> xyz=1.750 1.250 0.018 rpy=0 0 0
- joint joint_tile_7_9: origin xyz=1.350 0.750 0.027 rpy=0 0 0 -> xyz=2.250 1.250 0.017 rpy=0 0 0
- joint joint_tile_8_0: origin xyz=-1.350 1.050 0.026 rpy=0 0 0 -> xyz=-2.250 1.750 0.020 rpy=0 0 0
- joint joint_tile_8_1: origin xyz=-1.050 1.050 0.008 rpy=0 0 0 -> xyz=-1.750 1.750 0.008 rpy=0 0 0
- joint joint_tile_8_2: origin xyz=-0.750 1.050 0.018 rpy=0 0 0 -> xyz=-1.250 1.750 0.013 rpy=0 0 0
- joint joint_tile_8_3: origin xyz=-0.450 1.050 0.034 rpy=0 0 0 -> xyz=-0.750 1.750 0.015 rpy=0 0 0
- joint joint_tile_8_4: origin xyz=-0.150 1.050 0.034 rpy=0 0 0 -> xyz=-0.250 1.750 0.016 rpy=0 0 0
- joint joint_tile_8_5: origin xyz=0.150 1.050 0.005 rpy=0 0 0 -> xyz=0.250 1.750 0.008 rpy=0 0 0
- joint joint_tile_8_6: origin xyz=0.450 1.050 0.025 rpy=0 0 0 -> xyz=0.750 1.750 0.011 rpy=0 0 0
- joint joint_tile_8_7: origin xyz=0.750 1.050 0.019 rpy=0 0 0 -> xyz=1.250 1.750 0.010 rpy=0 0 0
- joint joint_tile_8_8: origin xyz=1.050 1.050 0.006 rpy=0 0 0 -> xyz=1.750 1.750 0.008 rpy=0 0 0
- joint joint_tile_8_9: origin xyz=1.350 1.050 0.029 rpy=0 0 0 -> xyz=2.250 1.750 0.011 rpy=0 0 0
- joint joint_tile_9_0: origin xyz=-1.350 1.350 0.009 rpy=0 0 0 -> xyz=-2.250 2.250 0.006 rpy=0 0 0
- joint joint_tile_9_1: origin xyz=-1.050 1.350 0.015 rpy=0 0 0 -> xyz=-1.750 2.250 0.007 rpy=0 0 0
- joint joint_tile_9_2: origin xyz=-0.750 1.350 0.033 rpy=0 0 0 -> xyz=-1.250 2.250 0.008 rpy=0 0 0
- joint joint_tile_9_3: origin xyz=-0.450 1.350 0.020 rpy=0 0 0 -> xyz=-0.750 2.250 0.011 rpy=0 0 0
- joint joint_tile_9_4: origin xyz=-0.150 1.350 0.018 rpy=0 0 0 -> xyz=-0.250 2.250 0.006 rpy=0 0 0
- joint joint_tile_9_5: origin xyz=0.150 1.350 0.010 rpy=0 0 0 -> xyz=0.250 2.250 0.019 rpy=0 0 0
- joint joint_tile_9_6: origin xyz=0.450 1.350 0.027 rpy=0 0 0 -> xyz=0.750 2.250 0.009 rpy=0 0 0
- joint joint_tile_9_7: origin xyz=0.750 1.350 0.024 rpy=0 0 0 -> xyz=1.250 2.250 0.017 rpy=0 0 0
- joint joint_tile_9_8: origin xyz=1.050 1.350 0.020 rpy=0 0 0 -> xyz=1.750 2.250 0.011 rpy=0 0 0
- joint joint_tile_9_9: origin xyz=1.350 1.350 0.024 rpy=0 0 0 -> xyz=2.250 2.250 0.012 rpy=0 0 0
