Commit message: modify the obstacle.urdf

File: assets/obstacle.urdf (robot description, URDF)
Before this commit: robot obstacle_regions, 21 links, 20 joints
Links:
- added link region_100, mass 0.1; collision box size=0.15000000000000002 0.05 0.01; visual box size=0.15000000000000002 0.05 0.01
- added link region_101, mass 0.1; collision box size=0.05 0.1 0.01; visual box size=0.05 0.1 0.01
- added link region_102, mass 0.1; collision box size=0.05 0.05 0.01; visual box size=0.05 0.05 0.01
- added link region_103, mass 0.1; collision box size=0.05 0.1 0.01; visual box size=0.05 0.1 0.01
- added link region_104, mass 0.1; collision box size=0.15000000000000002 0.05 0.01; visual box size=0.15000000000000002 0.05 0.01
- added link region_105, mass 0.1; collision box size=0.05 0.05 0.01; visual box size=0.05 0.05 0.01
- added link region_106, mass 0.1; collision box size=0.15000000000000002 0.1 0.01; visual box size=0.15000000000000002 0.1 0.01
- added link region_107, mass 0.1; collision box size=0.05 0.05 0.01; visual box size=0.05 0.05 0.01
- added link region_108, mass 0.1; collision box size=0.15000000000000002 0.1 0.01; visual box size=0.15000000000000002 0.1 0.01
- added link region_109, mass 0.1; collision box size=0.05 0.1 0.01; visual box size=0.05 0.1 0.01
- added link region_110, mass 0.1; collision box size=0.1 0.1 0.01; visual box size=0.1 0.1 0.01
- added link region_111, mass 0.1; collision box size=0.15000000000000002 0.15000000000000002 0.01; visual box size=0.15000000000000002 0.15000000000000002 0.01
- added link region_112, mass 0.1; collision box size=0.05 0.15000000000000002 0.01; visual box size=0.05 0.15000000000000002 0.01
- added link region_113, mass 0.1; collision box size=0.1 0.05 0.01; visual box size=0.1 0.05 0.01
- added link region_114, mass 0.1; collision box size=0.15000000000000002 0.1 0.01; visual box size=0.15000000000000002 0.1 0.01
- added link region_115, mass 0.1; collision box size=0.05 0.1 0.01; visual box size=0.05 0.1 0.01
- added link region_116, mass 0.1; collision box size=0.05 0.05 0.01; visual box size=0.05 0.05 0.01
- added link region_117, mass 0.1; collision box size=0.1 0.1 0.01; visual box size=0.1 0.1 0.01
- added link region_118, mass 0.1; collision box size=0.05 0.05 0.01; visual box size=0.05 0.05 0.01
- added link region_119, mass 0.1; collision box size=0.15000000000000002 0.05 0.01; visual box size=0.15000000000000002 0.05 0.01
- added link region_120, mass 0.1; collision box size=0.1 0.15000000000000002 0.01; visual box size=0.1 0.15000000000000002 0.01
- added link region_121, mass 0.1; collision box size=0.05 0.1 0.01; visual box size=0.05 0.1 0.01
- added link region_122, mass 0.1; collision box size=0.05 0.15000000000000002 0.01; visual box size=0.05 0.15000000000000002 0.01
- added link region_123, mass 0.1; collision box size=0.1 0.1 0.01; visual box size=0.1 0.1 0.01
- added link region_124, mass 0.1; collision box size=0.1 0.05 0.01; visual box size=0.1 0.05 0.01
- added link region_125, mass 0.1; collision box size=0.05 0.1 0.01; visual box size=0.05 0.1 0.01
- added link region_126, mass 0.1; collision box size=0.05 0.05 0.01; visual box size=0.05 0.05 0.01
- added link region_127, mass 0.1; collision box size=0.15000000000000002 0.15000000000000002 0.01; visual box size=0.15000000000000002 0.15000000000000002 0.01
- added link region_128, mass 0.1; collision box size=0.15000000000000002 0.05 0.01; visual box size=0.15000000000000002 0.05 0.01
- added link region_129, mass 0.1; collision box size=0.15000000000000002 0.05 0.01; visual box size=0.15000000000000002 0.05 0.01
- added link region_130, mass 0.1; collision box size=0.05 0.05 0.01; visual box size=0.05 0.05 0.01
- added link region_131, mass 0.1; collision box size=0.1 0.05 0.01; visual box size=0.1 0.05 0.01
- added link region_132, mass 0.1; collision box size=0.05 0.1 0.01; visual box size=0.05 0.1 0.01
- added link region_133, mass 0.1; collision box size=0.05 0.05 0.01; visual box size=0.05 0.05 0.01
- added link region_134, mass 0.1; collision box size=0.15000000000000002 0.05 0.01; visual box size=0.15000000000000002 0.05 0.01
- added link region_135, mass 0.1; collision box size=0.05 0.15000000000000002 0.01; visual box size=0.05 0.15000000000000002 0.01
- added link region_136, mass 0.1; collision box size=0.1 0.05 0.01; visual box size=0.1 0.05 0.01
- added link region_137, mass 0.1; collision box size=0.1 0.05 0.01; visual box size=0.1 0.05 0.01
- added link region_138, mass 0.1; collision box size=0.15000000000000002 0.05 0.01; visual box size=0.15000000000000002 0.05 0.01
- added link region_139, mass 0.1; collision box size=0.1 0.05 0.01; visual box size=0.1 0.05 0.01
- added link region_140, mass 0.1; collision box size=0.1 0.05 0.01; visual box size=0.1 0.05 0.01
- added link region_141, mass 0.1; collision box size=0.05 0.1 0.01; visual box size=0.05 0.1 0.01
- added link region_142, mass 0.1; collision box size=0.05 0.05 0.01; visual box size=0.05 0.05 0.01
- added link region_143, mass 0.1; collision box size=0.1 0.05 0.01; visual box size=0.1 0.05 0.01
- added link region_144, mass 0.1; collision box size=0.1 0.1 0.01; visual box size=0.1 0.1 0.01
- added link region_145, mass 0.1; collision box size=0.1 0.05 0.01; visual box size=0.1 0.05 0.01
- added link region_146, mass 0.1; collision box size=0.05 0.05 0.01; visual box size=0.05 0.05 0.01
- added link region_147, mass 0.1; collision box size=0.05 0.1 0.01; visual box size=0.05 0.1 0.01
- added link region_148, mass 0.1; collision box size=0.05 0.15000000000000002 0.01; visual box size=0.05 0.15000000000000002 0.01
- added link region_149, mass 0.1; collision box size=0.05 0.05 0.01; visual box size=0.05 0.05 0.01
- added link region_20, mass 0.1; collision box size=0.1 0.05 0.01; visual box size=0.1 0.05 0.01
- added link region_21, mass 0.1; collision box size=0.15000000000000002 0.05 0.01; visual box size=0.15000000000000002 0.05 0.01
- added link region_22, mass 0.1; collision box size=0.05 0.15000000000000002 0.01; visual box size=0.05 0.15000000000000002 0.01
- added link region_23, mass 0.1; collision box size=0.1 0.1 0.01; visual box size=0.1 0.1 0.01
- added link region_24, mass 0.1; collision box size=0.05 0.1 0.01; visual box size=0.05 0.1 0.01
- added link region_25, mass 0.1; collision box size=0.15000000000000002 0.1 0.01; visual box size=0.15000000000000002 0.1 0.01
- added link region_26, mass 0.1; collision box size=0.05 0.15000000000000002 0.01; visual box size=0.05 0.15000000000000002 0.01
- added link region_27, mass 0.1; collision box size=0.05 0.1 0.01; visual box size=0.05 0.1 0.01
- added link region_28, mass 0.1; collision box size=0.15000000000000002 0.15000000000000002 0.01; visual box size=0.15000000000000002 0.15000000000000002 0.01
- added link region_29, mass 0.1; collision box size=0.1 0.15000000000000002 0.01; visual box size=0.1 0.15000000000000002 0.01
- added link region_30, mass 0.1; collision box size=0.15000000000000002 0.05 0.01; visual box size=0.15000000000000002 0.05 0.01
- added link region_31, mass 0.1; collision box size=0.15000000000000002 0.15000000000000002 0.01; visual box size=0.15000000000000002 0.15000000000000002 0.01
- added link region_32, mass 0.1; collision box size=0.15000000000000002 0.15000000000000002 0.01; visual box size=0.15000000000000002 0.15000000000000002 0.01
- added link region_33, mass 0.1; collision box size=0.05 0.1 0.01; visual box size=0.05 0.1 0.01
- added link region_34, mass 0.1; collision box size=0.05 0.15000000000000002 0.01; visual box size=0.05 0.15000000000000002 0.01
- added link region_35, mass 0.1; collision box size=0.05 0.15000000000000002 0.01; visual box size=0.05 0.15000000000000002 0.01
- added link region_36, mass 0.1; collision box size=0.05 0.05 0.01; visual box size=0.05 0.05 0.01
- added link region_37, mass 0.1; collision box size=0.1 0.1 0.01; visual box size=0.1 0.1 0.01
- added link region_38, mass 0.1; collision box size=0.05 0.05 0.01; visual box size=0.05 0.05 0.01
- added link region_39, mass 0.1; collision box size=0.1 0.15000000000000002 0.01; visual box size=0.1 0.15000000000000002 0.01
- added link region_40, mass 0.1; collision box size=0.05 0.1 0.01; visual box size=0.05 0.1 0.01
- added link region_41, mass 0.1; collision box size=0.05 0.15000000000000002 0.01; visual box size=0.05 0.15000000000000002 0.01
- added link region_42, mass 0.1; collision box size=0.15000000000000002 0.1 0.01; visual box size=0.15000000000000002 0.1 0.01
- added link region_43, mass 0.1; collision box size=0.05 0.15000000000000002 0.01; visual box size=0.05 0.15000000000000002 0.01
- added link region_44, mass 0.1; collision box size=0.1 0.05 0.01; visual box size=0.1 0.05 0.01
- added link region_45, mass 0.1; collision box size=0.15000000000000002 0.05 0.01; visual box size=0.15000000000000002 0.05 0.01
- added link region_46, mass 0.1; collision box size=0.05 0.05 0.01; visual box size=0.05 0.05 0.01
- added link region_47, mass 0.1; collision box size=0.05 0.05 0.01; visual box size=0.05 0.05 0.01
- added link region_48, mass 0.1; collision box size=0.1 0.15000000000000002 0.01; visual box size=0.1 0.15000000000000002 0.01
- added link region_49, mass 0.1; collision box size=0.05 0.1 0.01; visual box size=0.05 0.1 0.01
- added link region_50, mass 0.1; collision box size=0.05 0.1 0.01; visual box size=0.05 0.1 0.01
- added link region_51, mass 0.1; collision box size=0.1 0.15000000000000002 0.01; visual box size=0.1 0.15000000000000002 0.01
- added link region_52, mass 0.1; collision box size=0.1 0.05 0.01; visual box size=0.1 0.05 0.01
- added link region_53, mass 0.1; collision box size=0.05 0.05 0.01; visual box size=0.05 0.05 0.01
- added link region_54, mass 0.1; collision box size=0.1 0.05 0.01; visual box size=0.1 0.05 0.01
- added link region_55, mass 0.1; collision box size=0.05 0.1 0.01; visual box size=0.05 0.1 0.01
- added link region_56, mass 0.1; collision box size=0.05 0.1 0.01; visual box size=0.05 0.1 0.01
- added link region_57, mass 0.1; collision box size=0.1 0.1 0.01; visual box size=0.1 0.1 0.01
- added link region_58, mass 0.1; collision box size=0.1 0.05 0.01; visual box size=0.1 0.05 0.01
- added link region_59, mass 0.1; collision box size=0.15000000000000002 0.05 0.01; visual box size=0.15000000000000002 0.05 0.01
- added link region_60, mass 0.1; collision box size=0.05 0.15000000000000002 0.01; visual box size=0.05 0.15000000000000002 0.01
- added link region_61, mass 0.1; collision box size=0.1 0.05 0.01; visual box size=0.1 0.05 0.01
- added link region_62, mass 0.1; collision box size=0.1 0.1 0.01; visual box size=0.1 0.1 0.01
- added link region_63, mass 0.1; collision box size=0.05 0.1 0.01; visual box size=0.05 0.1 0.01
- added link region_64, mass 0.1; collision box size=0.05 0.15000000000000002 0.01; visual box size=0.05 0.15000000000000002 0.01
- added link region_65, mass 0.1; collision box size=0.15000000000000002 0.1 0.01; visual box size=0.15000000000000002 0.1 0.01
- added link region_66, mass 0.1; collision box size=0.15000000000000002 0.15000000000000002 0.01; visual box size=0.15000000000000002 0.15000000000000002 0.01
- added link region_67, mass 0.1; collision box size=0.1 0.15000000000000002 0.01; visual box size=0.1 0.15000000000000002 0.01
- added link region_68, mass 0.1; collision box size=0.05 0.05 0.01; visual box size=0.05 0.05 0.01
- added link region_69, mass 0.1; collision box size=0.05 0.15000000000000002 0.01; visual box size=0.05 0.15000000000000002 0.01
- added link region_70, mass 0.1; collision box size=0.05 0.05 0.01; visual box size=0.05 0.05 0.01
- added link region_71, mass 0.1; collision box size=0.15000000000000002 0.05 0.01; visual box size=0.15000000000000002 0.05 0.01
- added link region_72, mass 0.1; collision box size=0.05 0.15000000000000002 0.01; visual box size=0.05 0.15000000000000002 0.01
- added link region_73, mass 0.1; collision box size=0.1 0.05 0.01; visual box size=0.1 0.05 0.01
- added link region_74, mass 0.1; collision box size=0.05 0.15000000000000002 0.01; visual box size=0.05 0.15000000000000002 0.01
- added link region_75, mass 0.1; collision box size=0.1 0.05 0.01; visual box size=0.1 0.05 0.01
- added link region_76, mass 0.1; collision box size=0.15000000000000002 0.05 0.01; visual box size=0.15000000000000002 0.05 0.01
- added link region_77, mass 0.1; collision box size=0.15000000000000002 0.15000000000000002 0.01; visual box size=0.15000000000000002 0.15000000000000002 0.01
- added link region_78, mass 0.1; collision box size=0.1 0.15000000000000002 0.01; visual box size=0.1 0.15000000000000002 0.01
- added link region_79, mass 0.1; collision box size=0.05 0.1 0.01; visual box size=0.05 0.1 0.01
- added link region_80, mass 0.1; collision box size=0.05 0.15000000000000002 0.01; visual box size=0.05 0.15000000000000002 0.01
- added link region_81, mass 0.1; collision box size=0.1 0.05 0.01; visual box size=0.1 0.05 0.01
- added link region_82, mass 0.1; collision box size=0.1 0.1 0.01; visual box size=0.1 0.1 0.01
- added link region_83, mass 0.1; collision box size=0.1 0.05 0.01; visual box size=0.1 0.05 0.01
- added link region_84, mass 0.1; collision box size=0.1 0.05 0.01; visual box size=0.1 0.05 0.01
- added link region_85, mass 0.1; collision box size=0.05 0.05 0.01; visual box size=0.05 0.05 0.01
- added link region_86, mass 0.1; collision box size=0.1 0.15000000000000002 0.01; visual box size=0.1 0.15000000000000002 0.01
- added link region_87, mass 0.1; collision box size=0.05 0.1 0.01; visual box size=0.05 0.1 0.01
- added link region_88, mass 0.1; collision box size=0.05 0.05 0.01; visual box size=0.05 0.05 0.01
- added link region_89, mass 0.1; collision box size=0.1 0.05 0.01; visual box size=0.1 0.05 0.01
- added link region_90, mass 0.1; collision box size=0.05 0.05 0.01; visual box size=0.05 0.05 0.01
- added link region_91, mass 0.1; collision box size=0.15000000000000002 0.1 0.01; visual box size=0.15000000000000002 0.1 0.01
- added link region_92, mass 0.1; collision box size=0.1 0.05 0.01; visual box size=0.1 0.05 0.01
- added link region_93, mass 0.1; collision box size=0.15000000000000002 0.05 0.01; visual box size=0.15000000000000002 0.05 0.01
- added link region_94, mass 0.1; collision box size=0.15000000000000002 0.1 0.01; visual box size=0.15000000000000002 0.1 0.01
- added link region_95, mass 0.1; collision box size=0.05 0.05 0.01; visual box size=0.05 0.05 0.01
- added link region_96, mass 0.1; collision box size=0.05 0.05 0.01; visual box size=0.05 0.05 0.01
- added link region_97, mass 0.1; collision box size=0.1 0.05 0.01; visual box size=0.1 0.05 0.01
- added link region_98, mass 0.1; collision box size=0.05 0.05 0.01; visual box size=0.05 0.05 0.01
- added link region_99, mass 0.1; collision box size=0.15000000000000002 0.15000000000000002 0.01; visual box size=0.15000000000000002 0.15000000000000002 0.01
- link region_0: geometry collision box size=0.15000000000000002 0.1 0.01; visual box size=0.15000000000000002 0.1 0.01
- link region_1: geometry collision box size=0.05 0.15000000000000002 0.01; visual box size=0.05 0.15000000000000002 0.01
- link region_10: geometry collision box size=0.1 0.1 0.01; visual box size=0.1 0.1 0.01
- link region_11: geometry collision box size=0.1 0.1 0.01; visual box size=0.1 0.1 0.01
- link region_12: geometry collision box size=0.15000000000000002 0.15000000000000002 0.01; visual box size=0.15000000000000002 0.15000000000000002 0.01
- link region_13: geometry collision box size=0.15000000000000002 0.05 0.01; visual box size=0.15000000000000002 0.05 0.01
- link region_15: geometry collision box size=0.15000000000000002 0.1 0.01; visual box size=0.15000000000000002 0.1 0.01
- link region_16: geometry collision box size=0.1 0.1 0.01; visual box size=0.1 0.1 0.01
- link region_17: geometry collision box size=0.05 0.05 0.01; visual box size=0.05 0.05 0.01
- link region_18: geometry collision box size=0.05 0.15000000000000002 0.01; visual box size=0.05 0.15000000000000002 0.01
- link region_19: geometry collision box size=0.05 0.1 0.01; visual box size=0.05 0.1 0.01
- link region_2: geometry collision box size=0.1 0.15000000000000002 0.01; visual box size=0.1 0.15000000000000002 0.01
- link region_3: geometry collision box size=0.05 0.15000000000000002 0.01; visual box size=0.05 0.15000000000000002 0.01
- link region_4: geometry collision box size=0.05 0.15000000000000002 0.01; visual box size=0.05 0.15000000000000002 0.01
- link region_5: geometry collision box size=0.15000000000000002 0.15000000000000002 0.01; visual box size=0.15000000000000002 0.15000000000000002 0.01
- link region_6: geometry collision box size=0.1 0.1 0.01; visual box size=0.1 0.1 0.01
- link region_7: geometry collision box size=0.05 0.15000000000000002 0.01; visual box size=0.05 0.15000000000000002 0.01
- link region_8: geometry collision box size=0.05 0.15000000000000002 0.01; visual box size=0.05 0.15000000000000002 0.01
- link region_9: geometry collision box size=0.05 0.15000000000000002 0.01; visual box size=0.05 0.15000000000000002 0.01
Joints:
- added joint region_100_joint: type fixed, parent base_link, child region_100, origin xyz=-0.41380501382722246 -1.6562398136935186 0.005 rpy=0 0 0
- added joint region_101_joint: type fixed, parent base_link, child region_101, origin xyz=2.2863577215344266 -0.24680026482622952 0.005 rpy=0 0 0
- added joint region_102_joint: type fixed, parent base_link, child region_102, origin xyz=1.7334634428819324 0.3944168399157202 0.005 rpy=0 0 0
- added joint region_103_joint: type fixed, parent base_link, child region_103, origin xyz=-0.10320196124795578 0.1315067172592519 0.005 rpy=0 0 0
- added joint region_104_joint: type fixed, parent base_link, child region_104, origin xyz=-1.7356151890384006 1.9459938043157603 0.005 rpy=0 0 0
- added joint region_105_joint: type fixed, parent base_link, child region_105, origin xyz=0.26700116990870093 0.2774072601696469 0.005 rpy=0 0 0
- added joint region_106_joint: type fixed, parent base_link, child region_106, origin xyz=-1.818979413690202 0.32945439361586226 0.005 rpy=0 0 0
- added joint region_107_joint: type fixed, parent base_link, child region_107, origin xyz=0.5697556363466321 -1.12240142503248 0.005 rpy=0 0 0
- added joint region_108_joint: type fixed, parent base_link, child region_108, origin xyz=0.111109900568517 0.46415826648667924 0.005 rpy=0 0 0
- added joint region_109_joint: type fixed, parent base_link, child region_109, origin xyz=0.6391693775192508 0.5528257989467082 0.005 rpy=0 0 0
- added joint region_110_joint: type fixed, parent base_link, child region_110, origin xyz=1.203518238013681 1.7936095258072373 0.005 rpy=0 0 0
- added joint region_111_joint: type fixed, parent base_link, child region_111, origin xyz=-1.4797787237204072 -0.35613511038517776 0.005 rpy=0 0 0
- added joint region_112_joint: type fixed, parent base_link, child region_112, origin xyz=-0.5980776145485409 -0.09147164861493984 0.005 rpy=0 0 0
- added joint region_113_joint: type fixed, parent base_link, child region_113, origin xyz=1.957555035645668 -1.1098835084351 0.005 rpy=0 0 0
- added joint region_114_joint: type fixed, parent base_link, child region_114, origin xyz=-1.7526970181746082 1.6822827089681458 0.005 rpy=0 0 0
- added joint region_115_joint: type fixed, parent base_link, child region_115, origin xyz=0.037708178324881825 -0.6276319669266142 0.005 rpy=0 0 0
- added joint region_116_joint: type fixed, parent base_link, child region_116, origin xyz=1.4232883083413461 -0.7167451875054542 0.005 rpy=0 0 0
- added joint region_117_joint: type fixed, parent base_link, child region_117, origin xyz=-0.8065552095331481 -1.0256863923634225 0.005 rpy=0 0 0
- added joint region_118_joint: type fixed, parent base_link, child region_118, origin xyz=1.4290175543065762 0.6475378161326901 0.005 rpy=0 0 0
- added joint region_119_joint: type fixed, parent base_link, child region_119, origin xyz=-1.5173256047204977 0.760093828494647 0.005 rpy=0 0 0
- added joint region_120_joint: type fixed, parent base_link, child region_120, origin xyz=0.2477524691607278 -1.5358276048489439 0.005 rpy=0 0 0
- added joint region_121_joint: type fixed, parent base_link, child region_121, origin xyz=1.5907926535828958 -1.2307122052009511 0.005 rpy=0 0 0
- added joint region_122_joint: type fixed, parent base_link, child region_122, origin xyz=0.7392196413380439 0.13693045549943683 0.005 rpy=0 0 0
- added joint region_123_joint: type fixed, parent base_link, child region_123, origin xyz=-2.1150134029985987 -0.7373071132309506 0.005 rpy=0 0 0
- added joint region_124_joint: type fixed, parent base_link, child region_124, origin xyz=0.9025342045030098 1.6741590206614627 0.005 rpy=0 0 0
- added joint region_125_joint: type fixed, parent base_link, child region_125, origin xyz=0.5443233211536107 -0.9413268958781191 0.005 rpy=0 0 0
- added joint region_126_joint: type fixed, parent base_link, child region_126, origin xyz=1.280941788517795 0.40320947491210557 0.005 rpy=0 0 0
- added joint region_127_joint: type fixed, parent base_link, child region_127, origin xyz=1.3566008551962017 -0.21598176175059658 0.005 rpy=0 0 0
- added joint region_128_joint: type fixed, parent base_link, child region_128, origin xyz=1.688701783062128 -0.07758991861512698 0.005 rpy=0 0 0
- added joint region_129_joint: type fixed, parent base_link, child region_129, origin xyz=-0.48125414172837067 -1.0413391066413613 0.005 rpy=0 0 0
- added joint region_130_joint: type fixed, parent base_link, child region_130, origin xyz=1.6392760011238554 -0.8773223846025897 0.005 rpy=0 0 0
- added joint region_131_joint: type fixed, parent base_link, child region_131, origin xyz=1.993556378215592 -0.10903856828773084 0.005 rpy=0 0 0
- added joint region_132_joint: type fixed, parent base_link, child region_132, origin xyz=0.5049118173746727 1.5392719891757873 0.005 rpy=0 0 0
- added joint region_133_joint: type fixed, parent base_link, child region_133, origin xyz=-0.9882489749159689 1.6034347366728636 0.005 rpy=0 0 0
- added joint region_134_joint: type fixed, parent base_link, child region_134, origin xyz=-0.995332281150533 1.329354961783762 0.005 rpy=0 0 0
- added joint region_135_joint: type fixed, parent base_link, child region_135, origin xyz=-1.5671864306417005 -1.2935144481812446 0.005 rpy=0 0 0
- added joint region_136_joint: type fixed, parent base_link, child region_136, origin xyz=0.20512680831280905 -0.8122160998895458 0.005 rpy=0 0 0
- added joint region_137_joint: type fixed, parent base_link, child region_137, origin xyz=-2.4042873126307147 -0.5242682972363031 0.005 rpy=0 0 0
- added joint region_138_joint: type fixed, parent base_link, child region_138, origin xyz=1.083794328075545 -1.625080268927502 0.005 rpy=0 0 0
- added joint region_139_joint: type fixed, parent base_link, child region_139, origin xyz=-1.4410330628566819 0.16497038698469035 0.005 rpy=0 0 0
- added joint region_140_joint: type fixed, parent base_link, child region_140, origin xyz=-0.9306487367312675 1.0428335163746514 0.005 rpy=0 0 0
- added joint region_141_joint: type fixed, parent base_link, child region_141, origin xyz=0.38520713691043706 -1.0824507656027045 0.005 rpy=0 0 0
- added joint region_142_joint: type fixed, parent base_link, child region_142, origin xyz=1.2588152306821803 1.0578409274025313 0.005 rpy=0 0 0
- added joint region_143_joint: type fixed, parent base_link, child region_143, origin xyz=2.406751415218518 -1.5850083959796661 0.005 rpy=0 0 0
- added joint region_144_joint: type fixed, parent base_link, child region_144, origin xyz=-1.3313765236394064 -0.7139556529555906 0.005 rpy=0 0 0
- added joint region_145_joint: type fixed, parent base_link, child region_145, origin xyz=-0.1703056669501679 -0.05771075780016233 0.005 rpy=0 0 0
- added joint region_146_joint: type fixed, parent base_link, child region_146, origin xyz=-0.7582171147853487 -1.2068906215165618 0.005 rpy=0 0 0
- added joint region_147_joint: type fixed, parent base_link, child region_147, origin xyz=0.02885161496029287 -0.3414240293000632 0.005 rpy=0 0 0
- added joint region_148_joint: type fixed, parent base_link, child region_148, origin xyz=-2.468417201272848 1.8187596066242127 0.005 rpy=0 0 0
- added joint region_149_joint: type fixed, parent base_link, child region_149, origin xyz=1.5454367830917501 -1.9660476695529496 0.005 rpy=0 0 0
- added joint region_20_joint: type fixed, parent base_link, child region_20, origin xyz=-0.2870898071444543 0.6318234376661689 0.005 rpy=0 0 0
- added joint region_21_joint: type fixed, parent base_link, child region_21, origin xyz=2.1951410176148585 1.0699813410618022 0.005 rpy=0 0 0
- added joint region_22_joint: type fixed, parent base_link, child region_22, origin xyz=-2.0269901571574276 -0.051684826840601605 0.005 rpy=0 0 0
- added joint region_23_joint: type fixed, parent base_link, child region_23, origin xyz=-1.1831244135161256 0.4765929740607526 0.005 rpy=0 0 0
- added joint region_24_joint: type fixed, parent base_link, child region_24, origin xyz=1.8791223647832744 1.6188694035816868 0.005 rpy=0 0 0
- added joint region_25_joint: type fixed, parent base_link, child region_25, origin xyz=1.774266126803914 -1.750738116195325 0.005 rpy=0 0 0
- added joint region_26_joint: type fixed, parent base_link, child region_26, origin xyz=-1.2695839014124937 -0.0742951131200329 0.005 rpy=0 0 0
- added joint region_27_joint: type fixed, parent base_link, child region_27, origin xyz=-1.6572024616605234 0.11967804747207866 0.005 rpy=0 0 0
- added joint region_28_joint: type fixed, parent base_link, child region_28, origin xyz=-0.8052679691395659 0.744266201871842 0.005 rpy=0 0 0
- added joint region_29_joint: type fixed, parent base_link, child region_29, origin xyz=0.8144132504630357 -1.7441599136204124 0.005 rpy=0 0 0
- added joint region_30_joint: type fixed, parent base_link, child region_30, origin xyz=2.059194322431325 -0.34153939152632473 0.005 rpy=0 0 0
- added joint region_31_joint: type fixed, parent base_link, child region_31, origin xyz=-1.3799099578281606 1.6398928343635966 0.005 rpy=0 0 0
- added joint region_32_joint: type fixed, parent base_link, child region_32, origin xyz=0.5645756103920068 0.9843269994782617 0.005 rpy=0 0 0
- added joint region_33_joint: type fixed, parent base_link, child region_33, origin xyz=0.8844400780686446 1.4399043903055717 0.005 rpy=0 0 0
- added joint region_34_joint: type fixed, parent base_link, child region_34, origin xyz=-1.6077191439845522 -0.6483690753376123 0.005 rpy=0 0 0
- added joint region_35_joint: type fixed, parent base_link, child region_35, origin xyz=0.006284578929824036 1.9055797643157453 0.005 rpy=0 0 0
- added joint region_36_joint: type fixed, parent base_link, child region_36, origin xyz=1.0942838523083416 -1.3185377262170657 0.005 rpy=0 0 0
- added joint region_37_joint: type fixed, parent base_link, child region_37, origin xyz=-1.3716245120040185 -1.4779204992186092 0.005 rpy=0 0 0
- added joint region_38_joint: type fixed, parent base_link, child region_38, origin xyz=-0.5506395783443454 1.7753027111256259 0.005 rpy=0 0 0
- added joint region_39_joint: type fixed, parent base_link, child region_39, origin xyz=-1.6527183426961938 -0.9877719494530246 0.005 rpy=0 0 0
- added joint region_40_joint: type fixed, parent base_link, child region_40, origin xyz=-0.9027725534162878 -0.17878527107624853 0.005 rpy=0 0 0
- added joint region_41_joint: type fixed, parent base_link, child region_41, origin xyz=1.053580599808293 1.0429151120638682 0.005 rpy=0 0 0
- added joint region_42_joint: type fixed, parent base_link, child region_42, origin xyz=0.6963004695099397 1.9121980701703585 0.005 rpy=0 0 0
- added joint region_43_joint: type fixed, parent base_link, child region_43, origin xyz=0.43284766463540825 1.2417052754312996 0.005 rpy=0 0 0
- added joint region_44_joint: type fixed, parent base_link, child region_44, origin xyz=2.070248308604616 -0.8562035750803976 0.005 rpy=0 0 0
- added joint region_45_joint: type fixed, parent base_link, child region_45, origin xyz=0.8669192628862037 -1.3407285957883472 0.005 rpy=0 0 0
- added joint region_46_joint: type fixed, parent base_link, child region_46, origin xyz=0.8754868354679868 -0.5251249263585482 0.005 rpy=0 0 0
- added joint region_47_joint: type fixed, parent base_link, child region_47, origin xyz=-2.2751923449079228 1.4995786468460697 0.005 rpy=0 0 0
- added joint region_48_joint: type fixed, parent base_link, child region_48, origin xyz=-0.9794808031850932 -1.5361637473264311 0.005 rpy=0 0 0
- added joint region_49_joint: type fixed, parent base_link, child region_49, origin xyz=-0.7695514135420063 1.2187725237543083 0.005 rpy=0 0 0
- added joint region_50_joint: type fixed, parent base_link, child region_50, origin xyz=-1.1481361542499233 -0.7212940648085733 0.005 rpy=0 0 0
- added joint region_51_joint: type fixed, parent base_link, child region_51, origin xyz=2.067141265325981 1.584954506736966 0.005 rpy=0 0 0
- added joint region_52_joint: type fixed, parent base_link, child region_52, origin xyz=0.8218049774150997 -0.32627439202594277 0.005 rpy=0 0 0
- added joint region_53_joint: type fixed, parent base_link, child region_53, origin xyz=0.5026012653519163 -0.7085321818860184 0.005 rpy=0 0 0
- added joint region_54_joint: type fixed, parent base_link, child region_54, origin xyz=-0.8848560544824142 0.49032020884989747 0.005 rpy=0 0 0
- added joint region_55_joint: type fixed, parent base_link, child region_55, origin xyz=1.114745968574589 -0.8855031349949247 0.005 rpy=0 0 0
- added joint region_56_joint: type fixed, parent base_link, child region_56, origin xyz=-0.6909232244065704 -1.4069004336325204 0.005 rpy=0 0 0
- added joint region_57_joint: type fixed, parent base_link, child region_57, origin xyz=2.4322578997557684 -0.018430507648070193 0.005 rpy=0 0 0
- added joint region_58_joint: type fixed, parent base_link, child region_58, origin xyz=-0.8069320445608514 0.08649659986591862 0.005 rpy=0 0 0
- added joint region_59_joint: type fixed, parent base_link, child region_59, origin xyz=-0.32956072540432 0.9126616913890779 0.005 rpy=0 0 0
- added joint region_60_joint: type fixed, parent base_link, child region_60, origin xyz=0.5919910751818676 -0.3567668713972565 0.005 rpy=0 0 0
- added joint region_61_joint: type fixed, parent base_link, child region_61, origin xyz=-1.1861063968655077 0.8550700957416209 0.005 rpy=0 0 0
- added joint region_62_joint: type fixed, parent base_link, child region_62, origin xyz=-0.37615982188362684 0.005779365458504326 0.005 rpy=0 0 0
- added joint region_63_joint: type fixed, parent base_link, child region_63, origin xyz=-0.5365271477897458 0.5337505814871477 0.005 rpy=0 0 0
- added joint region_64_joint: type fixed, parent base_link, child region_64, origin xyz=2.469438657465723 -0.7936242929210169 0.005 rpy=0 0 0
- added joint region_65_joint: type fixed, parent base_link, child region_65, origin xyz=-2.2538151295701385 1.8471699587981805 0.005 rpy=0 0 0
- added joint region_66_joint: type fixed, parent base_link, child region_66, origin xyz=-0.579402882190917 -0.8360202527954776 0.005 rpy=0 0 0
- added joint region_67_joint: type fixed, parent base_link, child region_67, origin xyz=-2.2846943465570746 0.7219548625678329 0.005 rpy=0 0 0
- added joint region_68_joint: type fixed, parent base_link, child region_68, origin xyz=1.3827703023818514 1.8318073687664733 0.005 rpy=0 0 0
- added joint region_69_joint: type fixed, parent base_link, child region_69, origin xyz=0.8056818172681197 0.5837723106973365 0.005 rpy=0 0 0
- added joint region_70_joint: type fixed, parent base_link, child region_70, origin xyz=1.6399733950818147 -0.7033851798360644 0.005 rpy=0 0 0
- added joint region_71_joint: type fixed, parent base_link, child region_71, origin xyz=-0.5069188493427834 -1.8897008104715265 0.005 rpy=0 0 0
- added joint region_72_joint: type fixed, parent base_link, child region_72, origin xyz=1.7533675757573652 1.8446563566204404 0.005 rpy=0 0 0
- added joint region_73_joint: type fixed, parent base_link, child region_73, origin xyz=1.9070649360563623 0.6023778831532969 0.005 rpy=0 0 0
- added joint region_74_joint: type fixed, parent base_link, child region_74, origin xyz=2.1929283439910687 0.5376538428200286 0.005 rpy=0 0 0
- added joint region_75_joint: type fixed, parent base_link, child region_75, origin xyz=0.11164036788883402 1.6368965686951467 0.005 rpy=0 0 0
- added joint region_76_joint: type fixed, parent base_link, child region_76, origin xyz=-2.186816965233744 -1.0502969232319495 0.005 rpy=0 0 0
- added joint region_77_joint: type fixed, parent base_link, child region_77, origin xyz=-2.389201121772726 1.0659819663012828 0.005 rpy=0 0 0
- added joint region_78_joint: type fixed, parent base_link, child region_78, origin xyz=-2.2166903520948296 0.3269932864216658 0.005 rpy=0 0 0
- added joint region_79_joint: type fixed, parent base_link, child region_79, origin xyz=-1.1672767453632433 -1.8591386945750772 0.005 rpy=0 0 0
- added joint region_80_joint: type fixed, parent base_link, child region_80, origin xyz=1.4040598824174122 -1.2762682078932663 0.005 rpy=0 0 0
- added joint region_81_joint: type fixed, parent base_link, child region_81, origin xyz=1.4601308983642234 1.6784999020023639 0.005 rpy=0 0 0
- added joint region_82_joint: type fixed, parent base_link, child region_82, origin xyz=-0.2634913185582137 1.1050781947404151 0.005 rpy=0 0 0
- added joint region_83_joint: type fixed, parent base_link, child region_83, origin xyz=0.4650988479986604 -0.052444841282901056 0.005 rpy=0 0 0
- added joint region_84_joint: type fixed, parent base_link, child region_84, origin xyz=-0.3360092470342311 1.7264562129586452 0.005 rpy=0 0 0
- added joint region_85_joint: type fixed, parent base_link, child region_85, origin xyz=-0.12364711815491658 -0.37270627456178707 0.005 rpy=0 0 0
- added joint region_86_joint: type fixed, parent base_link, child region_86, origin xyz=-2.205246034348261 -1.9060238267199212 0.005 rpy=0 0 0
- added joint region_87_joint: type fixed, parent base_link, child region_87, origin xyz=1.810545095218104 -0.6118777579063495 0.005 rpy=0 0 0
- added joint region_88_joint: type fixed, parent base_link, child region_88, origin xyz=2.4493803706110233 -1.2157207573202609 0.005 rpy=0 0 0
- added joint region_89_joint: type fixed, parent base_link, child region_89, origin xyz=-0.5359360131498059 1.3685942648273053 0.005 rpy=0 0 0
- added joint region_90_joint: type fixed, parent base_link, child region_90, origin xyz=-1.9349918548218756 1.2454997571536817 0.005 rpy=0 0 0
- added joint region_91_joint: type fixed, parent base_link, child region_91, origin xyz=1.6938929394065774 0.955838245144391 0.005 rpy=0 0 0
- added joint region_92_joint: type fixed, parent base_link, child region_92, origin xyz=0.13575458278689867 -1.8158671178970294 0.005 rpy=0 0 0
- added joint region_93_joint: type fixed, parent base_link, child region_93, origin xyz=-1.2870526611130864 -0.9272353006147829 0.005 rpy=0 0 0
- added joint region_94_joint: type fixed, parent base_link, child region_94, origin xyz=1.1735534490250559 0.07235717426436405 0.005 rpy=0 0 0
- added joint region_95_joint: type fixed, parent base_link, child region_95, origin xyz=0.21109540260649462 -0.2293885666734532 0.005 rpy=0 0 0
- added joint region_96_joint: type fixed, parent base_link, child region_96, origin xyz=0.13337792254496028 -1.0495239608088536 0.005 rpy=0 0 0
- added joint region_97_joint: type fixed, parent base_link, child region_97, origin xyz=2.1294830444240427 -1.3310346398104356 0.005 rpy=0 0 0
- added joint region_98_joint: type fixed, parent base_link, child region_98, origin xyz=-1.7798238409354508 -1.2960822884455705 0.005 rpy=0 0 0
- added joint region_99_joint: type fixed, parent base_link, child region_99, origin xyz=2.318016872029534 1.7806334317085741 0.005 rpy=0 0 0
- joint region_0_joint: origin xyz=-0.8228658824669033 0.2970202967603284 0.005 rpy=0 0 0 -> xyz=1.0496161458150173 0.4091980655360232 0.005 rpy=0 0 0
- joint region_10_joint: origin xyz=-1.2380924599004375 -1.4694298653724198 0.005 rpy=0 0 0 -> xyz=0.8143985616018496 0.8604271790039166 0.005 rpy=0 0 0
- joint region_11_joint: origin xyz=-0.3527062056192336 -0.8950300067902619 0.005 rpy=0 0 0 -> xyz=0.18796148970894633 -0.030179788485847903 0.005 rpy=0 0 0
- joint region_12_joint: origin xyz=-0.34639555527583954 -0.6519127426723278 0.005 rpy=0 0 0 -> xyz=-1.4427131714622292 1.1307224236599756 0.005 rpy=0 0 0
- joint region_13_joint: origin xyz=-1.492042635192996 -0.8679598231363963 0.005 rpy=0 0 0 -> xyz=-1.6039932459650053 -0.08448589499257708 0.005 rpy=0 0 0
- joint region_14_joint: origin xyz=-0.26662814461005624 1.2136982041261146 0.005 rpy=0 0 0 -> xyz=1.4016167117250449 -0.9271417065039178 0.005 rpy=0 0 0
- joint region_15_joint: origin xyz=-1.3997914175876212 -1.0594638751260952 0.005 rpy=0 0 0 -> xyz=2.170931993951865 0.2118678666021956 0.005 rpy=0 0 0
- joint region_16_joint: origin xyz=-0.5225213152828576 -0.21755603520671807 0.005 rpy=0 0 0 -> xyz=-1.1787370943376645 0.1763992938223482 0.005 rpy=0 0 0
- joint region_17_joint: origin xyz=-0.18436745849645653 -0.07298733541731006 0.005 rpy=0 0 0 -> xyz=2.458322558238218 -0.33961855174616584 0.005 rpy=0 0 0
- joint region_18_joint: origin xyz=-1.317019053004927 -1.3745104903572247 0.005 rpy=0 0 0 -> xyz=1.9365808359161578 0.9959421592823401 0.005 rpy=0 0 0
- joint region_19_joint: origin xyz=-1.160451025581084 1.3807975352807942 0.005 rpy=0 0 0 -> xyz=-0.6017377860226694 -0.567108045842939 0.005 rpy=0 0 0
- joint region_1_joint: origin xyz=-1.4463999764607096 -1.335211312663783 0.005 rpy=0 0 0 -> xyz=-0.07718492768030627 -1.3381399393968956 0.005 rpy=0 0 0
- joint region_2_joint: origin xyz=-0.5268917392209771 0.5650549582762614 0.005 rpy=0 0 0 -> xyz=-2.429538961763818 0.29523802876945426 0.005 rpy=0 0 0
- joint region_3_joint: origin xyz=-0.2423229522714807 0.3227594477371025 0.005 rpy=0 0 0 -> xyz=1.750278867091981 -0.30901559646482135 0.005 rpy=0 0 0
- joint region_4_joint: origin xyz=-1.2169555827110359 0.9581296200978158 0.005 rpy=0 0 0 -> xyz=-2.237551908332745 -1.5631957992003638 0.005 rpy=0 0 0
- joint region_5_joint: origin xyz=-0.023867198412260482 0.02025921219826965 0.005 rpy=0 0 0 -> xyz=1.4949519770920165 0.4439711253185421 0.005 rpy=0 0 0
- joint region_6_joint: origin xyz=-0.09831351557546708 -0.9668602254822234 0.005 rpy=0 0 0 -> xyz=-1.4839857279560702 -1.938458604155132 0.005 rpy=0 0 0
- joint region_7_joint: origin xyz=-1.0170739318958122 0.6056938463996526 0.005 rpy=0 0 0 -> xyz=-1.2045548366234595 -0.41398807849779606 0.005 rpy=0 0 0
- joint region_8_joint: origin xyz=-0.03500015362269249 1.0712547536022026 0.005 rpy=0 0 0 -> xyz=1.3288480638836409 -1.6835712359955606 0.005 rpy=0 0 0
- joint region_9_joint: origin xyz=-1.4842845276466972 -0.9952547598313957 0.005 rpy=0 0 0 -> xyz=-2.1459829919803126 -0.38890536454756286 0.005 rpy=0 0 0
